Commit message: Added tf frames and Meshes for CSO

File: simulator/cso_gnc_sim/res/models/world.urdf (robot description, URDF)
Before this commit: robot cso_visualization, 3 links, 2 joints
Links:
- link cso: geometry visual mesh filename=package://cso_gnc_sim/res/meshes/cso-mesh.stl scale=0.001 0.001 0.001

Commit message: added TF publisher configuration, texture, adjusted tf_publisher and rviz templates. NOTE: Texture still wronggit status

File: simulator/cso_gnc_sim/res/models/world.urdf (robot description, URDF)
Before this commit: robot cso_visualization, 3 links, 2 joints
Links:
- link teme: geometry visual mesh filename=package://cso_gnc_sim/res/meshes/earth-mesh.stl scale=1 1 1

Commit message: Feature/space tf rework

File: simulator/cso_gnc_sim/res/models/world.urdf (robot description, URDF)
Before this commit: robot cso_visualization, 3 links, 2 joints
Links:
- removed link cso
- added link chaser; visual mesh filename=package://cso_gnc_sim/res/meshes/cso-mesh.stl scale=0.001 0.001 0.001
Joints:
- joint cso2teme: child cso -> chaser

Commit message: Change layout of propagator builder and therefore changed also the layout of corresponding yaml files. Also increased the size of the cad model in the visualization.
Signed-off-by: Christian Lanegger <clanegge@student.ethz.ch>

File: simulator/cso_gnc_sim/res/models/world.urdf (robot description, URDF)
Before this commit: robot cso_visualization, 3 links, 2 joints
Links:
- link chaser: geometry visual mesh filename=package://cso_gnc_sim/res/meshes/cso-mesh.stl scale=1 1 1
- link target: geometry visual box size=1 1 1

Commit message: Cleanup, scenario visualizer

File: simulator/cso_gnc_sim/res/models/world.urdf (robot description, URDF)
Before this commit: robot cso_visualization, 3 links, 2 joints
Links:
- removed link teme
- added link J2K; visual mesh filename=package://cso_gnc_sim/res/meshes/earth-mesh.stl scale=1 1 1
Joints:
- removed joint cso2teme
- removed joint target2teme
- added joint cso2J2K: type fixed, parent J2K, child cso, origin xyz=0 0 0 
- added joint target2J2K: type fixed, parent J2K, child target, origin xyz=7000000 0 0 
