Commit message: Changes in Swisscube definition and visualization
Signed-off-by: michael.pantic <mpantic@student.ethz.ch>

File: rospace_simulator/res/models/world_cubesat.urdf (robot description, URDF)
Before this commit: robot cso_visualization, 2 links, 1 joints
Links:
- link swisscube: geometry visual box size=0.1 0.1 0.1
