Commit message: Corrected fixed frame name (J2K)

File: rospace_simulator/res/models/world.urdf (robot description, URDF)
Before this commit: robot cso_visualization, 3 links, 2 joints
Links:
- removed link cso
- added link chaser; visual mesh filename=package://rospace_simulator/res/meshes/cso-mesh.stl scale=1 1 1
- link J2K: geometry visual mesh filename=package://rospace_simulator/res/meshes/earth-mesh.stl scale=1 1 1
Joints:
- removed joint cso2J2K
- added joint chaser2J2K: type fixed, parent J2K, child chaser, origin xyz=0 0 0 

Commit message: Added a blue cube to rviz for SwissCube and a thrusting class which thrust all the time to the builder.
Signed-off-by: Christian Lanegger <clanegge@student.ethz.ch>

File: rospace_simulator/res/models/world.urdf (robot description, URDF)
Before this commit: robot cso_visualization, 3 links, 2 joints
Links:
- link target: geometry visual box size=100 100 100

Commit message: just visual changes to tf_publisher and fixed the Earth finally!!!!!
Signed-off-by: Christian Lanegger <clanegge@student.ethz.ch>

File: rospace_simulator/res/models/world.urdf (robot description, URDF)
Before this commit: robot cso_visualization, 3 links, 2 joints
Links:
- link J2K: geometry visual mesh filename=package://rospace_simulator/res/meshes/earth.DAE scale=637100 637100 637100
