Commit message: Changed structure of world.urdf files according to new .launch structure.
Xacro files have been implemented which now created the corresponding urdf
file needed for visualization. There are three main types of xacro files.
	1) <Scenarion>.urdf.xacro: loads planets and spacecrafts for the
				   scenario and creates the correct links.
	2) spacecraft.urdf.xacro: holds all spacecraft templates (currently
				  for chaser and target)
	3) planet.urdf.xacro: holds all planet templates (currently for Earth)

The xacro files load the configuration file with all spacecraft names and
therefore if the spacecraft names should change the urdf file is also updated
accordingly. I believe that is quite neat.

The new structure is now working completely. Next step is to updated all
existing launch files to scenarios, improve propagation parse to allow
different types of input coordinates as well as update and implement new
tests.

Signed-off-by: Christian Lanegger <christian.lanegger@epfl.ch>

File: rospace_simulator/res/worlds/world.urdf (robot description, URDF)
Before this commit: robot cso_visualization, 3 links, 2 joints
Joints:
- joint target2J2K: origin xyz=7000000 0 0  -> xyz=0 0 0 
