Commit message: Scenarios are now called Missions. Each of those can now have multiple scenarios.
The so-called scenarios (which was used before) has now
been renamed to (the more logical) mission. Every mission now can
have multiple scenarios (initial conditions). This was done so
that the different scenarios from the monte carlo testing
of the relative navigation filter can be ported to new structure.

The difference now is that the simulator.launch file requires two
arguments which are a mission and its corresponding scenario.

Signed-off-by: Christian Lanegger <christian.lanegger@epfl.ch>

File: rospace_simulator/res/worlds/world_dzhanibekov.urdf.xacro (robot description, xacro)
@@ -1,8 +1,9 @@
 <?xml version="1.0"?>
 <robot xmlns:xacro="http://www.ros.org/wiki/xacro" name="dzhanibekov">
+    <xacro:arg name="scenario" default="False"/>
     <xacro:include filename="$(find rospace_simulator)/res/urdf/spacecrafts.urdf.xacro" />
     <xacro:include filename="$(find rospace_simulator)/res/urdf/planets.urdf.xacro" />
     <!-- Location of Scenario Configuation File -->
-    <xacro:property name="config_location" value="$(find rospace_simulator)/cfg/Scenarios/dzhanibekov.yaml" />
+    <xacro:property name="config_location" value="$(find rospace_simulator)/cfg/Scenarios/dzhanibekov/$(arg scenario).yaml" />
     <!-- Initialize/Load parameters necessary for model creation -->
     <xacro:property name="inertial_frame" value="J2K"/>

File: rospace_simulator/res/worlds/world_envisat_mission.urdf.xacro (robot description, xacro)
@@ -1,8 +1,9 @@
 <?xml version="1.0"?>
 <robot xmlns:xacro="http://www.ros.org/wiki/xacro" name="envisat_mission">
+    <xacro:arg name="scenario" default="False"/>
     <xacro:include filename="$(find rospace_simulator)/res/urdf/spacecrafts.urdf.xacro" />
     <xacro:include filename="$(find rospace_simulator)/res/urdf/planets.urdf.xacro" />
     <xacro:property name="inertial_frame" value="J2K"/>
-    <xacro:property name="config_location" value="$(find rospace_simulator)/cfg/Scenarios/envisat_mission.yaml" />
+    <xacro:property name="config_location" value="$(find rospace_simulator)/cfg/Scenarios/envisat_mission/$(arg scenario).yaml" />
     <xacro:property name="namespace" value="${load_yaml(config_location)}"/>
     <!-- Load Planets -->

File: rospace_simulator/res/worlds/world_swisscube_mission.urdf.xacro (robot description, xacro)
@@ -1,8 +1,9 @@
 <?xml version="1.0"?>
 <robot xmlns:xacro="http://www.ros.org/wiki/xacro" name="swisscube_mission">
+    <xacro:arg name="scenario" default="False"/>
     <xacro:include filename="$(find rospace_simulator)/res/urdf/spacecrafts.urdf.xacro" />
     <xacro:include filename="$(find rospace_simulator)/res/urdf/planets.urdf.xacro" />
     <xacro:property name="inertial_frame" value="J2K"/>
-    <xacro:property name="config_location" value="$(find rospace_simulator)/cfg/Scenarios/swisscube_mission.yaml" />
+    <xacro:property name="config_location" value="$(find rospace_simulator)/cfg/Scenarios/swisscube_mission/$(arg scenario).yaml" />
     <xacro:property name="namespace" value="${load_yaml(config_location)}"/>
     <!-- Load Planets -->
