Commit message: Modified the dzhanibekov simulation so that it runs with new framework.
A T_handle spacecraft has been created which is used in the dzhanibekov
scenario and which also loads the beatiful T-handle mesh
created Michael.

Additionally a small bug in the satellite_tf launch file has been fixed
where a remapping was missing and therefore no lvlh frame was being
published.

Signed-off-by: Christian Lanegger <christian.lanegger@epfl.ch>

File: rospace_simulator/res/urdf/spacecrafts.urdf.xacro (robot description, xacro)
@@ -10,4 +10,7 @@
         <xacro:if value="${'target' in namespace}">
             <xacro:target_spacecraft namespace="${namespace}" joint_parent="${joint_parent}"/>
+        </xacro:if>
+        <xacro:if value="${'t_handle' in namespace.lower()}">
+            <xacro:T_handle_spacecraft namespace="${namespace}" joint_parent="${joint_parent}"/>
         </xacro:if>
     </xacro:macro>
@@ -44,5 +47,22 @@
             <parent link="${joint_parent}"/>
             <child link="${namespace}"/>
-        </joint>>
+        </joint>
+    </xacro:macro>
+    <xacro:macro name="T_handle_spacecraft" params="namespace joint_parent">
+        <link name="${namespace}">
+            <visual>
+                <geometry>
+                    <mesh filename="${meshes_location}/T_handle/T_handle.stl" scale="1 1 1">
+                    </mesh>
+                </geometry>
+                <material name="LightGrey" />
+                <origin rpy="0 0 0" xyz="0 -0.057977 0"/>
+            </visual>
+        </link>
+        <joint name="${namespace}2${joint_parent}" type="fixed">
+            <parent link="${joint_parent}"/>
+            <child link="${namespace}"/>
+            <origin xyz="7000000 0 0 "/>
+        </joint>
     </xacro:macro>
 </robot>

Commit message: Changed the files for the SwissCube simulation so that it works with the new framework.
This has been done exactly the same as in the commits before
so there is nothing new to report  except that it works
as before under the new structure.

Signed-off-by: Christian Lanegger <christian.lanegger@epfl.ch>

File: rospace_simulator/res/urdf/spacecrafts.urdf.xacro (robot description, xacro)
@@ -3,14 +3,17 @@
     <xacro:include filename="$(find rospace_simulator)/res/urdf/materials.urdf.xacro" />
     <xacro:property name="meshes_location" value="package://rospace_simulator/res/meshes"/>
-    <!-- Search for finding correct spacecraft template -->
+    <!-- Search for finding correct spacecraft template. Search is case insensitive. -->
     <xacro:macro name="load_spacecraft" params="namespace joint_parent">
-        <xacro:if value="${'chaser' in namespace}">
+        <xacro:if value="${'chaser' in namespace.lower()}">
             <xacro:chaser_spacecraft namespace="${namespace}" joint_parent="${joint_parent}"/>
         </xacro:if>
-        <xacro:if value="${'target' in namespace}">
+        <xacro:if value="${'target' in namespace.lower()}">
             <xacro:target_spacecraft namespace="${namespace}" joint_parent="${joint_parent}"/>
         </xacro:if>
         <xacro:if value="${'t_handle' in namespace.lower()}">
             <xacro:T_handle_spacecraft namespace="${namespace}" joint_parent="${joint_parent}"/>
+        </xacro:if>
+        <xacro:if value="${'swisscube' in namespace.lower()}">
+            <xacro:swisscube_spacecraft namespace="${namespace}" joint_parent="${joint_parent}" />
         </xacro:if>
     </xacro:macro>
@@ -66,3 +69,20 @@
         </joint>
     </xacro:macro>
+    <xacro:macro name="swisscube_spacecraft" params="namespace joint_parent">
+        <link name="${namespace}">
+            <visual>
+                <origin xyz="0.0 0.0 0.0" rpy="0.0 0.0 0.0" />
+                <geometry>
+                    <box size="0.1 0.1 0.1"/>
+                </geometry>
+                <material name="Grey" />
+                <origin rpy="0 0 0" xyz="0 0 0"/>
+            </visual>
+        </link>
+        <joint name="${namespace}2${joint_parent}" type="fixed">
+            <parent link="${joint_parent}"/>
+            <child link="${namespace}"/>
+            <origin xyz="7000000 0 0" rpy="0.0 0.0 0.0"/>
+        </joint>
+    </xacro:macro>
 </robot>

File: rospace_simulator/res/worlds/world_two.urdf (robot description, URDF)
Before this commit: robot dzhanibekov, 2 links, 1 joints
Links:
- removed link t_handle
- added link swisscube; visual box size=0.1 0.1 0.1
Joints:
- removed joint t_handle2J2K
- added joint swisscube2J2K: type fixed, parent joint_parent, child swisscube, origin xyz=7000000 0 0 rpy=0.0 0.0 0.0

Commit message: Fixed small bug in DipoleModel test and added EnviSat mission to scenarios.
The bug in the DipoleModel test was caused a wrong import. It was looking for
the module in the old package (propagator).

The EnviSat mission was added/updated so that it works with the new API. It also
was briefly tested and provides the same accuracy as under the old API.

Signed-off-by: Christian Lanegger <christian.lanegger@epfl.ch>

File: rospace_simulator/res/urdf/spacecrafts.urdf.xacro (robot description, xacro)
@@ -16,4 +16,7 @@
         <xacro:if value="${'swisscube' in namespace.lower()}">
             <xacro:swisscube_spacecraft namespace="${namespace}" joint_parent="${joint_parent}" />
+        </xacro:if>
+        <xacro:if value="${'envisat' in namespace.lower()}">
+            <xacro:envisat_spacecraft namespace="${namespace}" joint_parent="${joint_parent}" />
         </xacro:if>
     </xacro:macro>
@@ -86,3 +89,21 @@
         </joint>
     </xacro:macro>
+    <xacro:macro name="envisat_spacecraft" params="namespace joint_parent">
+        <link name="${namespace}">
+            <visual>
+                <origin xyz="0.0 0.0 0.0" rpy="0.0 0.0 0.0" />
+                <geometry>
+                    <mesh filename="${meshes_location}/envisat/ENVISAT.stl" scale="1 1 1">
+                    </mesh>
+                </geometry>
+                <material name="Grey" />
+                <origin rpy="0 0 0" xyz="0 0 0"/>
+            </visual>
+        </link>
+        <joint name="${namespace}2${joint_parent}" type="fixed">
+            <parent link="${joint_parent}"/>
+            <child link="${namespace}"/>
+            <origin xyz="7000000 0 0" rpy="0.0 0.0 0.0"/>
+        </joint>
+    </xacro:macro>
 </robot>

Commit message: Relative Navigation Filter ported to new core structure.
The filter now works with the new structure and so far two
scenarios have been added from the created experiments
(one close-range and one far-range). Additional can be easily
added by creating new scenario cfg files with the initial
conditions of the experiment.

Signed-off-by: Christian Lanegger <christian.lanegger@epfl.ch>

File: rospace_simulator/res/urdf/spacecrafts.urdf.xacro (robot description, xacro)
@@ -27,5 +27,5 @@
                 <origin xyz="0.0 0.0 0.0" rpy="0.0 0.0 0.0" />
                 <geometry>
-                    <mesh filename="${meshes_location}/cso/cso-mesh.stl" scale="1 1 1">
+                    <mesh filename="${meshes_location}/cso/cso-mesh.stl" scale="0.5 0.5 0.5">
                     </mesh>
                 </geometry>
